Commit message: ch5-9 Gazebo and ros2_control

File: ros2_ws/src/my_robot_description/urdf/arm.ros2_control.xacro (robot description, xacro)
@@ -3,10 +3,10 @@
     <ros2_control name="Arm" type="system">
         <hardware>
-            <!-- <plugin>mock_components/GenericSystem</plugin>
-            <param name="calculate_dynamics">true</param> -->
-            <plugin>arm_hardware/ArmHardwareInterface</plugin>
+            <plugin>mock_components/GenericSystem</plugin>
+            <param name="calculate_dynamics">true</param>
+            <!-- <plugin>arm_hardware/ArmHardwareInterface</plugin>
             <param name="joint1_motor_id">10</param>
             <param name="joint2_motor_id">20</param>
-            <param name="dynamixel_port">/dev/ttyUSB0</param>
+            <param name="dynamixel_port">/dev/ttyUSB0</param> -->
         </hardware>
         <joint name="arm_joint1">

File: ros2_ws/src/my_robot_description/urdf/arm.xacro (robot description, xacro)
@@ -16,4 +16,12 @@
             <material name="orange" />
         </visual>
+        <collision>
+            <geometry>
+                <box size="${arm_base_length} ${arm_base_width} ${arm_base_height}" />
+            </geometry>
+            <origin xyz="0 0 ${arm_base_height / 2.0}" rpy="0 0 0"/>
+        </collision>
+        <xacro:box_inertia m="0.5" x="${arm_base_length}" y="${arm_base_width}" z="${arm_base_height}"
+                            o_xyz="0 0 ${arm_base_height / 2.0}" o_rpy="0 0 0"/>
     </link>
     <link name="forearm_link">
@@ -25,4 +33,12 @@
             <material name="yellow" />
         </visual>
+        <collision>
+            <geometry>
+                <cylinder radius="${forearm_radius}" length="${forearm_length}" />
+            </geometry>
+            <origin xyz="0 0 ${forearm_length / 2.0}" rpy="0 0 0"/>
+        </collision>
+        <xacro:cylinder_inertia m="0.3" r="${forearm_radius}" l="${forearm_length}"
+                                o_xyz="0 0 ${forearm_length / 2.0}" o_rpy="0 0 0"/>
     </link>
     <link name="hand_link">
@@ -34,4 +50,12 @@
             <material name="orange" />
         </visual>
+        <collision>
+            <geometry>
+                <cylinder radius="${hand_radius}" length="${hand_length}" />
+            </geometry>
+            <origin xyz="0 0 ${hand_length / 2.0}" rpy="0 0 0"/>
+        </collision>
+        <xacro:cylinder_inertia m="0.3" r="${hand_radius}" l="${hand_length}"
+                                o_xyz="0 0 ${hand_length / 2.0}" o_rpy="0 0 0"/>
     </link>
     <joint name="arm_joint1" type="revolute">

File: ros2_ws/src/my_robot_description/urdf/common_properties.xacro (robot description, xacro)
@@ -13,3 +13,30 @@
         <color rgba="1 1 0 1" />
     </material>
+    <xacro:macro name="box_inertia" params="m x y z o_xyz o_rpy">
+        <inertial>
+            <mass value="${m}" />
+            <origin xyz="${o_xyz}" rpy="${o_rpy}" />
+            <inertia ixx="${(m/12) * (y*y + z*z)}" ixy="0" ixz="0"
+                     iyy="${(m/12) * (x*x + z*z)}" iyz="0"
+                     izz="${(m/12) * (x*x + y*y)}" />
+        </inertial>
+    </xacro:macro>
+    <xacro:macro name="cylinder_inertia" params="m r l o_xyz o_rpy">
+        <inertial>
+            <mass value="${m}" />
+            <origin xyz="${o_xyz}" rpy="${o_rpy}" />
+            <inertia ixx="${(m/12) * (3*r*r + l*l)}" ixy="0" ixz="0"
+                     iyy="${(m/12) * (3*r*r + l*l)}" iyz="0"
+                     izz="${(m/2) * (r*r)}" />
+        </inertial>
+    </xacro:macro>
+    <xacro:macro name="sphere_inertia" params="m r o_xyz o_rpy">
+        <inertial>
+            <mass value="${m}" />
+            <origin xyz="${o_xyz}" rpy="${o_rpy}" />
+            <inertia ixx="${(2/5) *m *r *r}" ixy="0" ixz="0"
+                     iyy="${(2/5) * m * r * r}" iyz="0"
+                     izz="${(2/5) * m * r * r}" />
+        </inertial>
+    </xacro:macro>
 </robot>

File: ros2_ws/src/my_robot_description/urdf/mobile_base.xacro (robot description, xacro)
@@ -15,4 +15,12 @@
             <material name="blue" />
         </visual>
+        <collision>
+            <geometry>
+                <box size="${base_length} ${base_width} ${base_height}" />
+            </geometry>
+            <origin xyz="0 0 ${base_height / 2.0}" rpy="0 0 0" />
+        </collision>
+        <xacro:box_inertia m="5.0" x="${base_length}" y="${base_width}" z="${base_height}"
+                        o_xyz="0 0 ${base_height / 2.0}" o_rpy="0 0 0"/>
     </link>
     <xacro:macro name="wheel_link" params="prefix">
@@ -25,4 +33,12 @@
                 <material name="grey" />
             </visual>
+            <collision>
+                <geometry>
+                    <sphere radius="${wheel_radius}" />
+                </geometry>
+                <origin xyz="0 0 0" rpy="0 0 0" />
+            </collision>
+            <xacro:cylinder_inertia m="1.0" r="${wheel_radius}" l="${wheel_length}"
+                                    o_xyz="0 0 0" o_rpy="${pi /2.0} 0 0"/>
         </link>
     </xacro:macro>
@@ -37,4 +53,12 @@
             <material name="grey" />
         </visual>
+        <collision>
+            <geometry>
+                <sphere radius="${wheel_radius / 2.0}" />
+            </geometry>
+            <origin xyz="0 0 0" rpy="0 0 0" />
+        </collision>
+        <xacro:sphere_inertia m="0.5" r="${wheel_radius / 2.0}"
+                              o_xyz="0 0 0" o_rpy="0 0 0"/>
     </link>
     <joint name="base_joint" type="fixed">
